File: MKB_01/mkb_01/mkb_01.kicad_pcb (KiCad board)
At the start: 2 copper layers, 310 x 120 mm, 381 parts, among them J1 USB_C_Receptacle_USB2.0, J2 SW_Push, K1 SW_Push, M1 SW_Push, P1 SW_Push, Q1 SW_Push, Q2 BSP318, Q3 BSP318, T1 SW_Push, U1 LD1117S33TR_SOT223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

Commit message: routing optimizations
Routing:
- net PB0: track 373.5 -> 361.3 mm, vias 3 -> 2
- net CAPS_LIGHT: track 51.6 -> 57.3 mm
- net GND: track 104.2 -> 101.9 mm, vias 29 -> 27
- net 5V: track 26.4 -> 25.1 mm
- net PA5: track 165.4 -> 166.7 mm
- net LED_GND: track 1719.2 -> 1720.2 mm
- net PA4: track 395.2 -> 396.0 mm
- net PB7: track 250.4 -> 249.6 mm
- net PB8: track 229.7 -> 228.9 mm
- net PB9: track 210.8 -> 210.0 mm
- net PB6: track 263.9 -> 263.1 mm
- net PB3: track 338.3 -> 337.6 mm
- net PB5: track 304.3 -> 303.5 mm
- net PB4: track 319.4 -> 318.7 mm

Commit message: ordered
Other:
- board text added: "MKB_01 75% V1 Nils Wittig 2021 Top"
- board text added: "https://github.com/NilsWittig/mkb_01"
